Commit message: sv

File: crx_description/urdf/crx.ros2_control.xacro (robot description, xacro)
@@ -2,10 +2,14 @@
 <robot xmlns:xacro="http://www.ros.org/wiki/xacro">
   <xacro:macro name="crx_ros2_control"
-  params="name
-  robot_ip:=10.11.31.111
-  use_mock_hardware:=false
-  read_only:=false
-  use_rmi:=false">
-  <!-- Read only parameter should allow to move the robot via manual guidance, jog, etc throu the TP, and makes available the /joint_states topic -->
+    params="
+      name
+      robot_ip:=10.11.31.111
+      use_mock_hardware:=false
+      read_only:=false
+      use_rmi:=false
+      prefix:=''
+    ">
+    <!-- Read only parameter should allow to move the robot via manual guidance, jog, etc
+         through the TP, and makes available the /joint_states topic -->
     <ros2_control name="${name}" type="system">
       <hardware>
@@ -21,13 +25,9 @@
         </xacro:unless>
       </hardware>
-      <joint name="J1">
+      <joint name="${prefix}J1">
         <command_interface name="position">
           <param name="min">{-2*pi}</param>
           <param name="max">{2*pi}</param>
         </command_interface>
-        <!-- <command_interface name="velocity">
-          <param name="min">-3.15</param>
-          <param name="max">3.15</param>
-        </command_interface> -->
         <state_interface name="position">
           <param name="initial_value">0.0</param>
@@ -35,13 +35,9 @@
         <state_interface name="velocity"/>
       </joint>
-      <joint name="J2">
+      <joint name="${prefix}J2">
         <command_interface name="position">
           <param name="min">{-2*pi}</param>
           <param name="max">{2*pi}</param>
         </command_interface>
-        <!-- <command_interface name="velocity">
-          <param name="min">-3.15</param>
-          <param name="max">3.15</param>
-        </command_interface> -->
         <state_interface name="position">
           <param name="initial_value">0.0</param>
@@ -49,13 +45,9 @@
         <state_interface name="velocity"/>
       </joint>
-      <joint name="J3">
+      <joint name="${prefix}J3">
         <command_interface name="position">
           <param name="min">{-pi}</param>
           <param name="max">{pi}</param>
         </command_interface>
-        <!-- <command_interface name="velocity">
-          <param name="min">-3.15</param>
-          <param name="max">3.15</param>
-        </command_interface> -->
         <state_interface name="position">
           <param name="initial_value">0.0</param>
@@ -63,13 +55,9 @@
         <state_interface name="velocity"/>
       </joint>
-      <joint name="J4">
+      <joint name="${prefix}J4">
         <command_interface name="position">
           <param name="min">{-2*pi}</param>
           <param name="max">{2*pi}</param>
         </command_interface>
-        <!-- <command_interface name="velocity">
-          <param name="min">-3.2</param>
-          <param name="max">3.2</param>
-        </command_interface> -->
         <state_interface name="position">
           <param name="initial_value">0.0</param>
@@ -77,13 +65,9 @@
         <state_interface name="velocity"/>
       </joint>
-      <joint name="J5">
+      <joint name="${prefix}J5">
         <command_interface name="position">
           <param name="min">{-2*pi}</param>
           <param name="max">{2*pi}</param>
         </command_interface>
-        <!-- <command_interface name="velocity">
-          <param name="min">-3.2</param>
-          <param name="max">3.2</param>
-        </command_interface> -->
         <state_interface name="position">
           <param name="initial_value">0.0</param>
@@ -91,13 +75,9 @@
         <state_interface name="velocity"/>
       </joint>
-      <joint name="J6">
+      <joint name="${prefix}J6">
         <command_interface name="position">
           <param name="min">{-2*pi}</param>
           <param name="max">{2*pi}</param>
         </command_interface>
-        <!-- <command_interface name="velocity">
-          <param name="min">-3.2</param>
-          <param name="max">3.2</param>
-        </command_interface> -->
         <state_interface name="position">
           <param name="initial_value">0.0</param>

File: crx_description/urdf/crx10ia_l/bimanual_crx10ia_l.xacro (robot description, xacro)
@@ -1,6 +1,4 @@
 <?xml version="1.0"?>
 <robot xmlns:xacro="http://www.ros.org/wiki/xacro" name="crx_bimanual">
-  <xacro:arg name="left_robot_type"  default="crx10ia_l"/>
-  <xacro:arg name="right_robot_type" default="crx10ia_l"/>
   <xacro:arg name="use_mock_hardware" default="false"/>
   <xacro:arg name="left_robot_ip"  default="192.168.1.100"/>
@@ -9,37 +7,32 @@
   <xacro:arg name="use_rmi" default="false"/>
   <xacro:arg name="gz" default="false"/>
-  <!-- base offset of right arm in left base frame -->
+  <!-- base offset of right arm in world -->
   <xacro:arg name="right_base_xyz" default="0.8 0.0 0.0"/>
   <xacro:arg name="right_base_rpy" default="0.0 0.0 0.0"/>
-  <link name="world"/>
-  <!-- Include your single-arm xacro macro (or file) -->
-  <xacro:include filename="$(find crx_description)/urdf/${left_robot_type}/${left_robot_type}.xacro"/>
-  <xacro:include filename="$(find crx_description)/urdf/${right_robot_type}/${right_robot_type}.xacro"/>
-  <!-- Left arm instance -->
-  <xacro:property name="left_prefix" value="left_"/>
-  <!-- IMPORTANT: your arm xacro must accept 'prefix' and optionally 'parent' -->
-  <xacro:crx_arm
-      prefix="${left_prefix}"
+  <!-- include the single-arm wrapper that forwards prefix/parent/origin_* -->
+  <xacro:include filename="$(find crx_description)/urdf/crx10ia_l/crx10ia_l.xacro"/>
+  <!-- Left arm -->
+  <xacro:crx10ia_l
+      prefix="left_"
       parent="world"
-      robot_type="${left_robot_type}"
-      use_mock_hardware="${use_mock_hardware}"
-      robot_ip="${left_robot_ip}"
-      read_only="${read_only}"
-      use_rmi="${use_rmi}"
-      gz="${gz}"
+      origin_xyz="0 0 0"
+      origin_rpy="0 0 0"
+      use_mock_hardware="$(arg use_mock_hardware)"
+      robot_ip="$(arg left_robot_ip)"
+      read_only="$(arg read_only)"
+      use_rmi="$(arg use_rmi)"
+      gz="$(arg gz)"
   />
-  <!-- Right arm instance -->
-  <xacro:property name="right_prefix" value="right_"/>
-  <xacro:crx_arm
-      prefix="${right_prefix}"
+  <!-- Right arm -->
+  <xacro:crx10ia_l
+      prefix="right_"
       parent="world"
-      origin_xyz="${right_base_xyz}"
-      origin_rpy="${right_base_rpy}"
-      robot_type="${right_robot_type}"
-      use_mock_hardware="${use_mock_hardware}"
-      robot_ip="${right_robot_ip}"
-      read_only="${read_only}"
-      use_rmi="${use_rmi}"
-      gz="${gz}"
+      origin_xyz="$(arg right_base_xyz)"
+      origin_rpy="$(arg right_base_rpy)"
+      use_mock_hardware="$(arg use_mock_hardware)"
+      robot_ip="$(arg right_robot_ip)"
+      read_only="$(arg read_only)"
+      use_rmi="$(arg use_rmi)"
+      gz="$(arg gz)"
   />
 </robot>

File: crx_description/urdf/crx10ia_l/crx10ia_l.urdf.xacro (robot description, xacro)
@@ -2,9 +2,17 @@
 <robot xmlns:xacro="http://wiki.ros.org/xacro">
   <xacro:macro name="crx10ia_l"
-              params="robot_ip:='10.11.31.121'
-              read_only:='false'
-              use_rmi:='false'
-              use_mock_hardware:=false
-              gz:=false">
+              params="
+                robot_ip:='10.11.31.121'
+                read_only:='false'
+                use_rmi:='false'
+                use_mock_hardware:=false
+                gz:=false
+                prefix:=''
+                parent:='world'
+                origin_xyz:='0 0 0'
+                origin_rpy:='0 0 0'
+              ">
+    <!-- If your composite URDF defines world already, this is harmless; otherwise add it at top-level -->
+    <!-- <link name="world"/> -->
     <xacro:if value="${gz}">
       <xacro:include filename="$(find crx_description)/urdf/crx.gazebo.xacro" />
@@ -13,33 +21,37 @@
     <xacro:unless value="${gz}">
       <xacro:include filename="$(find crx_description)/urdf/crx.ros2_control.xacro" />
-      <xacro:crx_ros2_control name="crx10ia_l"
-                use_mock_hardware="${use_mock_hardware}"
-                robot_ip="${robot_ip}"
-                read_only="${read_only}"
-                use_rmi="${use_rmi}" />
+      <!-- IMPORTANT: give unique ros2_control system name per arm -->
+      <xacro:crx_ros2_control
+          name="${prefix}crx10ia_l"
+          use_mock_hardware="${use_mock_hardware}"
+          robot_ip="${robot_ip}"
+          read_only="${read_only}"
+          use_rmi="${use_rmi}"
+          prefix="${prefix}"/>
+      <!-- ^ You may need to add 'prefix' support inside crx.ros2_control.xacro too (see section 3) -->
     </xacro:unless>
-    <material name="black">
+    <material name="${prefix}black">
       <color rgba="0 0 0 1.0"/>
     </material>
-    <material name="white">
+    <material name="${prefix}white">
       <color rgba="1.0 1.0 1.0 1.00"/>
     </material>
     <!-- links -->
-    <link name="base_link">
-      <visual>
-      	<origin xyz="0 0 0" rpy="0 0 0"/>
-      	<geometry>
-      	  <mesh filename="package://crx_description/meshes/crx10ia_l/visual/link_base.stl" scale="0.001 0.001 0.001"/>
-      	</geometry>
-      	<material name="black"/>
-      </visual>
-      <collision>
-      	<origin xyz="0 0 0" rpy="0 0 0"/>
-      	<geometry>
-      	  <mesh filename="package://crx_description/meshes/crx10ia_l/collision/link_base.stl" scale="0.001 0.001 0.001"/>
-      	</geometry>
-      </collision>
-    </link>
-    <link name="link_1">
+  <link name="${prefix}base_link">
+    <visual>
+        <origin xyz="0 0 0" rpy="0 0 0"/>
+        <geometry>
+            <mesh filename="package://crx_description/meshes/crx10ia_l/visual/link_base.stl" scale="0.001 0.001 0.001"/>
+        </geometry>
+        <material name="${prefix}black"/>
+    </visual>
+    <collision>
+     <origin xyz="0 0 0" rpy="0 0 0"/>
+      <geometry>
+       <mesh filename="package://crx_description/meshes/crx10ia_l/collision/link_base.stl" scale="0.001 0.001 0.001"/>
+      </geometry>
+    </collision>
+  </link>
+  <link name="${prefix}link_1">
       <visual>
         <origin xyz="0 0 0" rpy="0 0 0"/>
@@ -56,5 +68,5 @@
       </collision>
     </link>
-    <link name="link_2">
+    <link name="${prefix}link_2">
       <visual>
         <origin xyz="0 0 0" rpy="0 0 0"/>
@@ -62,5 +74,5 @@
           <mesh filename="package://crx_description/meshes/crx10ia_l/visual/link_2.stl" scale="0.001 0.001 0.001"/>
         </geometry>
-        <material name="white"/>
+        <material name="${prefix}white"/>
       </visual>
       <collision>
@@ -71,5 +83,5 @@
       </collision>
     </link>
-    <link name="link_3">
+    <link name="${prefix}link_3">
       <visual>
         <origin xyz="0 0 0" rpy="0 0 0"/>
@@ -77,5 +89,5 @@
           <mesh filename="package://crx_description/meshes/crx10ia_l/visual/link_3.stl" scale="0.001 0.001 0.001"/>
         </geometry>
-        <material name="white"/>
+        <material name="${prefix}white"/>
       </visual>
       <collision>
@@ -86,5 +98,5 @@
       </collision>
     </link>
-    <link name="link_4">
+    <link name="${prefix}link_4">
       <visual>
         <origin xyz="0 0 0" rpy="0 0 0"/>
@@ -92,5 +104,5 @@
           <mesh filename="package://crx_description/meshes/crx10ia_l/visual/link_4.stl" scale="0.001 0.001 0.001"/>
         </geometry>
-        <material name="white"/>
+        <material name="${prefix}white"/>
       </visual>
       <collision>
@@ -101,5 +113,5 @@
       </collision>
     </link>
-    <link name="link_5">
+    <link name="${prefix}link_5">
       <visual>
         <origin xyz="0 0 0" rpy="0 0 0"/>
@@ -107,5 +119,5 @@
           <mesh filename="package://crx_description/meshes/crx10ia_l/visual/link_5.stl" scale="0.001 0.001 0.001"/>
         </geometry>
-        <material name="white"/>
+        <material name="${prefix}white"/>
       </visual>
       <collision>
@@ -116,5 +128,5 @@
       </collision>
     </link>
-    <link name="link_6">
+    <link name="${prefix}link_6">
       <visual>
         <origin xyz="0 0 0" rpy="0 0 0"/>
@@ -122,5 +134,5 @@
           <mesh filename="package://crx_description/meshes/crx10ia_l/visual/link_6.stl" scale="0.001 0.001 0.001"/>
         </geometry>
-        <material name="black"/>
+        <material name="${prefix}black"/>
       </visual>
       <collision>
@@ -131,67 +143,73 @@
       </collision>
     </link>
+    <!-- NEW: mount this arm under 'parent' with pose -->
+    <joint name="${prefix}mount_joint" type="fixed">
+      <origin xyz="${origin_xyz}" rpy="${origin_rpy}"/>
+      <parent link="${parent}"/>
+      <child link="${prefix}base_link"/>
+    </joint>
     <!-- joints -->
-    <joint name="J1" type="revolute">
+    <joint name="${prefix}J1" type="revolute">
       <origin xyz="0 0 0.1277" rpy="0 0 0"/>
-      <parent link="base_link"/>
-      <child link="link_1"/>
+      <parent link="${prefix}base_link"/>
+      <child link="${prefix}link_1"/>
       <axis xyz="0 0 1"/>
       <limit lower="${-180 * pi / 180}" upper="${180 * pi / 180}" effort="0" velocity="${80 * pi / 120}"/>
     </joint>
-    <joint name="J2" type="revolute">
+    <joint name="${prefix}J2" type="revolute">
       <origin xyz="0 0 0.1173" rpy="0 0 0"/>
-      <parent link="link_1"/>
-      <child link="link_2"/>
+      <parent link="${prefix}link_1"/>
+      <child link="${prefix}link_2"/>
       <axis xyz="0 1 0"/>
       <limit lower="${-180 * pi / 180}" upper="${180 * pi / 180}" effort="0" velocity="${80 * pi / 120}"/>
     </joint>
-    <joint name="J3" type="revolute">
+    <joint name="${prefix}J3" type="revolute">
       <origin xyz="0 0 0.710" rpy="0 0 0"/>
-      <parent link="link_2"/>
-      <child link="link_3"/>
+      <parent link="${prefix}link_2"/>
+      <child link="${prefix}link_3"/>
       <axis xyz="0 -1 0"/>
       <limit lower="${-270 * pi / 180}" upper="${270 * pi / 180}" effort="0" velocity="${120 * pi / 180}"/>
     </joint>
-    <joint name="J4" type="revolute">
+    <joint name="${prefix}J4" type="revolute">
       <origin xyz="0.540 0 0" rpy="0 0 0"/>
-      <parent link="link_3"/>
-      <child link="link_4"/>
+      <parent link="${prefix}link_3"/>
+      <child link="${prefix}link_4"/>
       <axis xyz="-1 0 0"/>
       <limit lower="${-190 * pi / 180}" upper="${190 * pi / 180}" effort="0" velocity="${112 * pi / 180}"/>
     </joint>
-    <joint name="J5" type="revolute">
+    <joint name="${prefix}J5" type="revolute">
       <origin xyz="0 -0.150 0" rpy="0 0 0"/>
-      <parent link="link_4"/>
-      <child link="link_5"/>
+      <parent link="${prefix}link_4"/>
+      <child link="${prefix}link_5"/>
       <axis xyz="0 -1 0"/>
       <limit lower="${-180 * pi / 180}" upper="${180 * pi / 180}" effort="0" velocity="${90 * pi / 180}"/>
     </joint>
-    <joint name="J6" type="revolute">
+    <joint name="${prefix}J6" type="revolute">
       <origin xyz="0.160 0 0" rpy="0 0 0"/>
-      <parent link="link_5"/>
-      <child link="link_6"/>
+      <parent link="${prefix}link_5"/>
+      <child link="${prefix}link_6"/>
       <axis xyz="-1 0 0"/>
       <limit lower="${-225 * pi / 180}" upper="${225 * pi / 180}" effort="0" velocity="${112 * pi / 180}"/>
     </joint>
     <!-- fanuc world -->
-    <link name="fanuc_world" />
-    <joint name="base_link-fanuc_world" type="fixed">
+    <link name="${prefix}fanuc_world" />
+    <joint name="${prefix}base_link-fanuc_world" type="fixed">
       <origin xyz="0 0 0.245" rpy="0 0 0"/>
-      <parent link="base_link"/>
-      <child link="fanuc_world"/>
+      <parent link="${prefix}base_link"/>
+      <child link="${prefix}fanuc_world"/>
     </joint>
     <!-- flange -->
-    <link name="flange" />
-    <joint name="J6-flange" type="fixed">
+    <link name="${prefix}flange" />
+    <joint name="${prefix}J6-flange" type="fixed">
       <origin xyz="0 0 0" rpy="0 0 0" />
-      <parent link="link_6" />
-      <child link="flange" />
+      <parent link="${prefix}link_6" />
+      <child link="${prefix}flange" />
     </joint>
     <!-- tcp -->
-    <link name="tcp" />
-    <joint name="flange-tcp" type="fixed">
+    <link name="${prefix}tcp" />
+    <joint name="${prefix}flange-tcp" type="fixed">
       <origin xyz="0 0 0" rpy="0 ${pi/2} 0" />
-      <parent link="flange" />
-      <child link="tcp" />
+      <parent link="${prefix}flange" />
+      <child link="${prefix}tcp" />
     </joint>
   </xacro:macro>

File: crx_description/urdf/crx10ia_l/crx10ia_l.xacro (robot description, xacro)
@@ -1,4 +1,5 @@
 <?xml version="1.0"?>
 <robot name="crx10ia_l" xmlns:xacro="http://wiki.ros.org/xacro">
+  <link name="world"/>
   <xacro:arg name="use_mock_hardware" default="true" />
   <xacro:arg name="read_only" default="false" />
@@ -6,5 +7,20 @@
   <xacro:arg name="use_rmi" default="false" />
   <xacro:arg name="gz" default="false" />
+  <!-- NEW -->
+  <xacro:arg name="prefix" default=""/>
+  <xacro:arg name="parent" default="world"/>
+  <xacro:arg name="origin_xyz" default="0 0 0"/>
+  <xacro:arg name="origin_rpy" default="0 0 0"/>
   <xacro:include filename="$(find crx_description)/urdf/crx10ia_l/crx10ia_l.urdf.xacro"/>
-  <xacro:crx10ia_l use_mock_hardware="$(arg use_mock_hardware)" robot_ip="$(arg robot_ip)" read_only="$(arg read_only)" use_rmi="$(arg use_rmi)" gz="$(arg gz)" />
+  <xacro:crx10ia_l
+      use_mock_hardware="$(arg use_mock_hardware)"
+      robot_ip="$(arg robot_ip)"
+      read_only="$(arg read_only)"
+      use_rmi="$(arg use_rmi)"
+      gz="$(arg gz)"
+      prefix="$(arg prefix)"
+      parent="$(arg parent)"
+      origin_xyz="$(arg origin_xyz)"
+      origin_rpy="$(arg origin_rpy)"
+  />
 </robot>
