Commit message: Sv

File: crx_description/urdf/crx10ia_l/crx10ia_l.urdf.xacro (robot description, xacro)
@@ -155,5 +155,5 @@
       <child link="${prefix}link_1"/>
       <axis xyz="0 0 1"/>
-      <limit lower="${-180 * pi / 180}" upper="${180 * pi / 180}" effort="0" velocity="${80 * pi / 120}"/>
+      <limit lower="${-179.9 * pi / 190}" upper="${179.9 * pi / 190}" effort="0" velocity="${80 * pi / 120}"/>
     </joint>
     <joint name="${prefix}J2" type="revolute">
@@ -162,5 +162,5 @@
       <child link="${prefix}link_2"/>
       <axis xyz="0 1 0"/>
-      <limit lower="${-180 * pi / 180}" upper="${180 * pi / 180}" effort="0" velocity="${80 * pi / 120}"/>
+      <limit lower="${-179.9 * pi / 180}" upper="${179.9 * pi / 180}" effort="0" velocity="${80 * pi / 120}"/>
     </joint>
     <joint name="${prefix}J3" type="revolute">
@@ -183,5 +183,5 @@
       <child link="${prefix}link_5"/>
       <axis xyz="0 -1 0"/>
-      <limit lower="${-180 * pi / 180}" upper="${180 * pi / 180}" effort="0" velocity="${90 * pi / 180}"/>
+      <limit lower="${-179.9 * pi / 180}" upper="${179.9 * pi / 180}" effort="0" velocity="${90 * pi / 180}"/>
     </joint>
     <joint name="${prefix}J6" type="revolute">

File: crx_description/urdf/crx_bimanual/crx_bimanual.xacro (robot description, xacro)
@@ -20,5 +20,5 @@
       parent="world"
       origin_xyz="0 0 0"
-      origin_rpy="0 0 0 "
+      origin_rpy="-0.5239 0 1.57 "
   />
   <!-- Right arm -->
@@ -31,6 +31,6 @@
       prefix="right_"
       parent="world"
-      origin_xyz="0.3 -0.50 0"
-      origin_rpy="0 0 0 "
+      origin_xyz="0.350 0.0 0"
+      origin_rpy="0.5235988 0 1.57 "
   />
 </robot>
